Commit message: update coffeebot description

File: description/lidar.xacro (robot description, xacro)
@@ -1,24 +1,59 @@
 <?xml version="1.0"?>
-<robot xmlns:xacro="http://www.ros.org/wiki/xacro"  >
-    <joint name="lidar_joint" type="fixed">
+<robot xmlns:xacro="http://www.ros.org/wiki/xacro" >
+    <joint name="laser_joint" type="fixed">
         <parent link="chassis"/>
-        <child link="lidar_frame"/>
-        <origin xyz="0.1 0.0 0.2" rpy="0.0 0.0 0.0"/>
+        <child link="laser_frame"/>
+        <origin xyz="0.15 0 0.25" rpy="0 0 0"/>
     </joint>
-    <link name="lidar_frame">
+    <link name="laser_frame">
         <visual>
             <geometry>
-                <cylinder radius="0.05" length="0.1"/>
+                <cylinder radius="0.05" length="0.08"/>
             </geometry>
             <material name="yellow"/>
         </visual>
+        <visual>
+            <origin xyz="0 0 -0.05"/>
+            <geometry>
+                <cylinder radius="0.01" length="0.1"/>
+            </geometry>
+            <material name="black"/>
+        </visual>
         <collision>
             <geometry>
-                <cylinder radius="0.05" length="0.1"/>
+                <cylinder radius="0.05" length="0.08"/>
             </geometry>
         </collision>
-        <xacro:inertial_cylinder mass="0.1" radius="0.1" length="0.1">
-            <origin xyz="0.0 0.0 0.0" rpy="0.0 0.0 0.0"/>
+        <xacro:inertial_cylinder mass="0.1" length="0.08" radius="0.05">
+            <origin xyz="0 0 0" rpy="0 0 0"/>
         </xacro:inertial_cylinder>
     </link>
+    <gazebo reference="laser_frame">
+        <material>Gazebo/Yellow</material>
+        <sensor name="laser" type="ray">
+            <pose> 0 0 0 0 0 0 </pose>
+            <visualize>true</visualize>
+            <update_rate>10</update_rate>
+            <ray>
+                <scan>
+                    <horizontal>
+                        <samples>360</samples>
+                        <min_angle>-3.14</min_angle>
+                        <max_angle>3.14</max_angle>
+                    </horizontal>
+                </scan>
+                <range>
+                    <min>0.3</min>
+                    <max>12</max>
+                </range>
+            </ray>
+            <plugin name="laser_controller" filename="libgazebo_ros_ray_sensor.so">
+                <ros>
+                    <argument>~/out:=scan</argument>
+                </ros>
+                <output_type>sensor_msgs/LaserScan</output_type>
+                <frame_name>laser_frame</frame_name>
+            </plugin>
+        </sensor>
+    </gazebo>
 </robot>

File: description/robot_core.xacro (robot description, xacro)
@@ -37,5 +37,5 @@
             </geometry>
         </collision>
-        <xacro:inertial_box mass="0.5" x="0.5" y="0.5" z="0.2">
+        <xacro:inertial_box mass="1.0" x="0.5" y="0.5" z="0.2">
             <origin xyz="0.25 0.0 0.1" rpy="0.0 0.0 0.0"/>
         </xacro:inertial_box>
@@ -123,15 +123,16 @@
         <mu2 value="0.001"/>
     </gazebo>
-<!-- Left_Pole_Link
+<!-- Left_Pole_Link -->
 <joint name="left_pole_joint" type="fixed">
-    <parent link="left_wheel"/>
+    <parent link="chassis"/>
     <child link="left_pole"/>
-    <origin xyz="0.0 -0.05 0.2" rpy="0.0 0.0 0.0"/>
-    <!<axis xyz="0.0 0.0 1.0"/>
+    <origin xyz="0.3 0.2 0.7" rpy="0.0 0.0 0.0"/>
+    <!-- <axis xyz="0.0 0.0 1.0"/>  -->
 </joint>
 <link name="left_pole">
     <visual>
-        <geometry>
-            <cylinder radius="0.1" length="1.0"/>
+        <!-- <origin xyz="0.1 -0.2 0.7"/> -->
+        <geometry>
+            <cylinder radius="0.025" length="1.0"/>
         </geometry>
         <material name="white"/>
@@ -139,13 +140,94 @@
     <collision>
         <geometry>
-            <cylinder radius="0.1" length="0.05"/>
-        </geometry>
-    </collision>
-    <xacro:inertial_cylinder mass="0.1" radius="0.1" length="0.05">
+            <cylinder radius="0.025" length="1.0"/>
+        </geometry>
+    </collision>
+    <xacro:inertial_cylinder mass="0.2" radius="0.025" length="1.0">
         <origin xyz="0.0 0.0 0.0" rpy="0.0 0.0 0.0"/>
     </xacro:inertial_cylinder>
 </link>
-<gazebo reference="left_wheel">
+<gazebo reference="left_pole">
+    <material>Gazebo/White</material>
+</gazebo>
+<!-- Right_Pole_Link -->
+<joint name="right_pole_joint" type="fixed">
+    <parent link="chassis"/>
+    <child link="right_pole"/>
+    <origin xyz="0.3 -0.2 0.7" rpy="0.0 0.0 0.0"/>
+    <!-- <axis xyz="0.0 0.0 1.0"/>  -->
+</joint>
+<link name="right_pole">
+    <visual>
+        <!-- <origin xyz="0.1 0.2 0.7"/> -->
+        <geometry>
+            <cylinder radius="0.025" length="1.0"/>
+        </geometry>
+        <material name="white"/>
+    </visual>
+    <collision>
+        <geometry>
+            <cylinder radius="0.025" length="1.0"/>
+        </geometry>
+    </collision>
+    <xacro:inertial_cylinder mass="0.2" radius="0.025" length="1.0">
+        <origin xyz="0.0 0.0 0.0" rpy="0.0 0.0 0.0"/>
+    </xacro:inertial_cylinder>
+</link>
+<gazebo reference="right_pole">
+    <material>Gazebo/White</material>
+</gazebo>
+<!-- Panel_Link -->
+<joint name="panel_joint" type="fixed">
+    <parent link="chassis"/>
+    <child link="panel"/>
+    <origin xyz="0.15 0.0 1.1" />
+</joint>
+<link name="panel">
+    <visual>
+        <origin xyz="0.15 0.0 0.0" rpy="0.0 0.0 ${pi/2}"/>
+        <geometry>
+            <box size="0.35 0.015 0.2"/>
+        </geometry>
+        <material name="black"/>
+    </visual>
+    <collision>
+        <origin xyz="0.15 0 0.0" />
+        <geometry>
+            <box size="0.35 0.15 0.2"/>
+        </geometry>
+    </collision>
+    <xacro:inertial_box mass="0.2" x="0.35" y="0.15" z="0.2">
+        <origin xyz="0.0 0.0 0.0" rpy="0.0 0.0 0.0"/>
+    </xacro:inertial_box>
+</link>
+<gazebo reference="panel">
     <material>Gazebo/Black</material>
-</gazebo> -->
+</gazebo>
+<!-- Tray_Link -->
+<joint name="tray_joint" type="fixed">
+    <parent link="chassis"/>
+    <child link="tray_link"/>
+    <origin xyz="0.15 0.0 0.7" />
+</joint>
+<link name="tray_link">
+    <visual>
+        <origin xyz="0.0 0.0 0.0" rpy="0.0 0.0 0.0"/>
+        <geometry>
+            <box size="0.5 0.5 0.05"/>
+        </geometry>
+        <material name="white"/>
+    </visual>
+    <collision>
+        <origin xyz="0.0 0 0.0" />
+        <geometry>
+            <box size="0.5 0.5 0.05"/>
+        </geometry>
+    </collision>
+    <xacro:inertial_box mass="0.2" x="0.5" y="0.5" z="0.05">
+        <origin xyz="0.0 0.0 0.0" rpy="0.0 0.0 0.0"/>
+    </xacro:inertial_box>
+</link>
+<gazebo reference="tray_link">
+    <material>Gazebo/White</material>
+</gazebo>
 </robot>
