Commit message: build coffeebot on gazebo

File: description/robot_core.xacro (robot description, xacro)
@@ -38,4 +38,7 @@
         </xacro:inertial_box>
     </link>
+    <gazebo reference="chassis">
+        <material>Gazebo/White</material>
+    </gazebo>
 <!-- Left_wheel_link -->
     <joint name="left_wheel_joint" type="continuous">
@@ -61,4 +64,7 @@
         </xacro:inertial_cylinder>
     </link>
+    <gazebo reference="left_wheel">
+        <material>Gazebo/Black</material>
+    </gazebo>
 <!-- Right_wheel_link -->
     <joint name="right_wheel_joint" type="continuous">
@@ -84,4 +90,7 @@
         </xacro:inertial_cylinder>
     </link>
+    <gazebo reference="right_wheel">
+        <material>Gazebo/Black</material>
+    </gazebo>
 <!-- Caster_wheel_link -->
     <joint name="caster_wheel_joint" type="fixed">
@@ -106,3 +115,6 @@
         </xacro:inertial_sphere>
     </link>
+    <gazebo reference="caster_wheel">
+        <material>Gazebo/Black</material>
+    </gazebo>
 </robot>

Commit message: add lidar

File: description/robot_core.xacro (robot description, xacro)
@@ -10,4 +10,7 @@
     <material name="orange">
         <color rgba="1 0.3 0.1 1"/>
+    </material>
+    <material name="yellow">
+        <color rgba="1 1 0 1"/>
     </material>
 <!-- Base_link -->
@@ -117,4 +120,32 @@
     <gazebo reference="caster_wheel">
         <material>Gazebo/Black</material>
+        <mu1 value="0.001"/>
+        <mu2 value="0.001"/>
     </gazebo>
+<!-- Left_Pole_Link
+<joint name="left_pole_joint" type="fixed">
+    <parent link="left_wheel"/>
+    <child link="left_pole"/>
+    <origin xyz="0.0 -0.05 0.2" rpy="0.0 0.0 0.0"/>
+    <!<axis xyz="0.0 0.0 1.0"/>
+</joint>
+<link name="left_pole">
+    <visual>
+        <geometry>
+            <cylinder radius="0.1" length="1.0"/>
+        </geometry>
+        <material name="white"/>
+    </visual>
+    <collision>
+        <geometry>
+            <cylinder radius="0.1" length="0.05"/>
+        </geometry>
+    </collision>
+    <xacro:inertial_cylinder mass="0.1" radius="0.1" length="0.05">
+        <origin xyz="0.0 0.0 0.0" rpy="0.0 0.0 0.0"/>
+    </xacro:inertial_cylinder>
+</link>
+<gazebo reference="left_wheel">
+    <material>Gazebo/Black</material>
+</gazebo> -->
 </robot>

Commit message: slam

File: description/robot_core.xacro (robot description, xacro)
@@ -17,4 +17,12 @@
     <link name="base_link">
     </link>
+<!-- BASE_FOOTPRINT LINK -->
+<joint name="base_footprint_joint" type="fixed">
+    <parent link="base_link"/>
+    <child link="base_footprint"/>
+    <origin xyz="0 0 0" rpy="0 0 0"/>
+</joint>
+<link name="base_footprint">
+</link>
 <!-- Chassis_link -->
     <joint name="chassis_joint" type="fixed">
